File: PiScreen.sch (KiCad schematic (older format))
At the start: 4 parts, among them P1 M02X05, P2 M02X05

Commit message: v0.1 PCB revision
Parts:
- added P3: CONN_14, symbol CONN_14
- added P4, P5, P6: CONN_5, symbol CONN_5
- added SJ1, SJ2, SJ3, SJ4, SJ5, SJ6, SJ7, SJ8, SJ9: SJ, symbol SJ
Connections:
- net labels added: +3.3V, OLED2_~CS, OLED2_~RST, uSD2_CD, uSD2_~CS
- wire segments 58 -> 103
- no-connect marks 12 -> 0
Other:
- note added: "Jumpers for dual displays/reconfiguration"
- note added: "NB: On Rev 1 Pi\nPin 3 = GPIO 0\nPin 5 = GPIO 1\nPin 13 = GPIO 21"
- note added: "OLED Right-angle connector"
- note added: "OLED Vertical Connector\n"
- note added: "Protoshield Breakout Sections"
- note removed: "OLED Connectors\n"
- note removed: "Right-angle connector"
- moved on the sheet: JP1, P1, P2, R1
